File: MEB.kicad_pcb (KiCad board)
At the start: 2 copper layers, 49.8 x 49.8 mm, 45 parts, among them J1 171857-0003, J10 1x4 Header, J2 171856-0002, J3 171857-0003, J4 171856-0002, J5 Header, J6 171856-0002, J7 171857-0003, J8 171856-0004, J9 TLW-104-05-T-D, P1 MSP-EXP430G2ET Interface with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, Q1 2.1V, Q2 2N7000, Q3 2N7000, Q4 TP2104N3-G, SW1 FSM2JSMA, SW2 FSM2JSMA, U1 NCP1117LPST33T3G

Commit message: Began PCB Design
Parts:
- removed F1: 0466002.NRHF, AltiumImport:FP-0466-MFG
- removed G***: LOGO, LOGO
- removed J10: 1x4 Header, AltiumImport:1X4 HEADER
- removed P1: MSP-EXP430G2ET Interface with 1x3 Power Headers, AltiumImport:MSP-EXP430G2ET Interface Power
- added C10: 10n, Capacitor_SMD:C_0805_2012Metric_Pad1.18x1.45mm_HandSolder, F.Cu at (75.2, 100.9)
- added C11: 47p, Capacitor_SMD:C_0805_2012Metric_Pad1.18x1.45mm_HandSolder, F.Cu at (75.2, 103.9)
- added C12: 47p, Capacitor_SMD:C_0805_2012Metric_Pad1.18x1.45mm_HandSolder, F.Cu at (75.2, 106.9)
- added C4: 12.5p, Capacitor_SMD:C_0805_2012Metric_Pad1.18x1.45mm_HandSolder, F.Cu at (62.8, 126.4)
- added C5: 100n, Capacitor_SMD:C_0805_2012Metric_Pad1.18x1.45mm_HandSolder, F.Cu at (62.8, 129.4)
- added C6: 10u, Capacitor_SMD:CP_Elec_4x5.8, F.Cu at (69.1, 124.8)
- added C7: 100n, Capacitor_SMD:C_0805_2012Metric_Pad1.18x1.45mm_HandSolder, F.Cu at (75.2, 94.9)
- added C8: 100n, Capacitor_SMD:C_0805_2012Metric_Pad1.18x1.45mm_HandSolder, F.Cu at (75.2, 97.9)
- added C9: 4.7u, Capacitor_SMD:CP_Elec_4x5.8, F.Cu at (81.5, 103.0)
- added D4: 3.2V, AltiumImport:0805_A, F.Cu at (85.3, 86.6)
- added D5: 3.2V, AltiumImport:0805_A, F.Cu at (85.3, 89.4)
- added D6: 3.2V, AltiumImport:0805_A, F.Cu at (101.3, 137.1)
- added R10: 27, Resistor_SMD:R_0805_2012Metric_Pad1.20x1.40mm_HandSolder, F.Cu at (65.8, 92.6)
- added R22: 10k, Resistor_SMD:R_0805_2012Metric_Pad1.20x1.40mm_HandSolder, F.Cu at (65.8, 98.5)
- added R23: 10k, Resistor_SMD:R_0805_2012Metric_Pad1.20x1.40mm_HandSolder, F.Cu at (65.8, 101.5)
- added R24: 10k, Resistor_SMD:R_0805_2012Metric_Pad1.20x1.40mm_HandSolder, F.Cu at (65.8, 104.4)
- added R25: 200, Resistor_SMD:R_0805_2012Metric_Pad1.20x1.40mm_HandSolder, F.Cu at (92.3, 96.5)
- added R26: 20, Resistor_SMD:R_0805_2012Metric_Pad1.20x1.40mm_HandSolder, F.Cu at (96.7, 137.5)
- added R8: 0, Resistor_SMD:R_0805_2012Metric_Pad1.20x1.40mm_HandSolder, F.Cu at (65.8, 86.7)
- added R9: 27, Resistor_SMD:R_0805_2012Metric_Pad1.20x1.40mm_HandSolder, F.Cu at (65.8, 89.7)
- added U2: MSP430FR2355TPT, SWLib:PT0048A_N, F.Cu at (167.8, 99.8)
- added U3: FT230XS-R, SWLib:SOIC_30XS-R_FTD, F.Cu at (81.9, 96.7)
- added U4: PCT2075DP, Package_SO:TSSOP-8_3x3mm_P0.65mm, F.Cu at (102.5, 112.8)
- added Y1: 32768, Crystal:Crystal_AT310_D3.0mm_L10.0mm_Horizontal, F.Cu at (56.3, 111.8)
- C3: value 1uF -> 12.5p; footprint AltiumImport:FP-0603-L_1_6_0_1-W_0_8_0-IPC_A -> Capacitor_SMD:C_0805_2012Metric_Pad1.18x1.45mm_HandSolder
- J5: value Header -> 171856-0004; footprint AltiumImport:2x3 Header -> AltiumImport:SHDR4W99P0X254_1X4_1001X635X1105P
- J6: value 171856-0002 -> 171857-0003; footprint AltiumImport:SHDR2W99P0X254_1X2_493X635X818P -> AltiumImport:171857-0003
- J7: value 171857-0003 -> Conn_01x07; footprint AltiumImport:171857-0003 -> Connector_PinHeader_2.54mm:PinHeader_1x07_P2.54mm_Vertical
- J8: value 171856-0004 -> USB_B_Micro; footprint AltiumImport:SHDR4W99P0X254_1X4_1001X635X1105P -> Connector_USB:USB_Micro-B_GCT_USB3076-30-A
- R1, R11, R12, R2, R3, R4, R5, R6, R7: footprint AltiumImport:SMD-0805-RES -> Resistor_SMD:R_0805_2012Metric_Pad1.20x1.40mm_HandSolder
- R13, R14: value 4.7k -> 0; footprint AltiumImport:SMD-0805-RES -> Resistor_SMD:R_0805_2012Metric_Pad1.20x1.40mm_HandSolder
- R15: footprint AltiumImport:FP-RMCF0805-IPC_C -> Resistor_SMD:R_0805_2012Metric_Pad1.20x1.40mm_HandSolder
- R16: footprint AltiumImport:FP-RNCP0805-IPC_C -> Resistor_SMD:R_0805_2012Metric_Pad1.20x1.40mm_HandSolder
- R17, R18, R19, R20: value 47 -> 0; footprint AltiumImport:SMD-0805-RES -> Resistor_SMD:R_0805_2012Metric_Pad1.20x1.40mm_HandSolder
- R21: value 47 -> 10k; footprint AltiumImport:SMD-0805-RES -> Resistor_SMD:R_0805_2012Metric_Pad1.20x1.40mm_HandSolder
- moved R21 85.1 mm to (65.8, 95.6)
- moved C3 78.4 mm to (62.8, 123.4), turned to 0 degrees
- moved R11 76.3 mm to (96.7, 131.6), turned to 0 degrees
- moved D2 76.0 mm to (101.3, 131.5), turned to 0 degrees
- moved R5 69.9 mm to (92.3, 90.6), turned to 0 degrees
- moved R20 62.3 mm to (96.7, 126.7), turned to 0 degrees
- moved R6 58.9 mm to (92.3, 93.6), turned to 0 degrees
- moved R12 58.7 mm to (96.7, 134.6)
- moved D3 56.5 mm to (101.3, 134.3), turned to 0 degrees
- moved Q2 53.4 mm to (98.4, 92.5), turned to 0 degrees
- moved J9 53.3 mm to (179.5, 127.4), turned to 0 degrees
- moved R19 52.1 mm to (96.7, 123.7), turned to 0 degrees
- moved J6 51.3 mm to (131.2, 124.8), turned to -90 degrees
- moved J2 49.7 mm to (174.4, 84.2)
- moved R18 47.3 mm to (96.7, 120.8), turned to 0 degrees
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Connections:
- net /launchpad_interface/leak_out renamed /leak_sensor/leak_out
- net /system_SSR_control/SYS_SW renamed /Input Headers/SYS_OFF
- net Net-(Q2-D) renamed /Input Headers/KillSwitchB
- net Net-(Q4-Gate) renamed /Input Headers/leak_probe
- C3 pad 1: 3V3 -> Net-(U2-P2.6_MCLK_XOUT)
- F2 pad 2: 3V3 -> +3V3
- J3 pad 2: /system_SSR_control/SW_ARM -> unconnected-(J3-Pad2)
- J4 pad 1: Net-(F1-Pad2) -> +BATT
- J5 pad 1: Net-(J5-Pad1) -> /Output Headers/I2C_SCL
- J5 pad 2: GND -> /Output Headers/I2C_SDA
- J5 pad 3: Net-(J5-Pad3) -> GND
- J5 pad 4: Net-(J5-Pad4) -> +3V3
- J6 pad 1: V_BAT -> GND
- J6 pad 2: GND -> /Output Headers/LED_Strip
- J7 pad 2: /launchpad_interface/LED_strip -> +5V
- J7 pad 3: 5V -> Net-(J7-Pin_3)
- J8 pad 1: /SCL -> +5V
- J8 pad 2: /SDA -> Net-(J8-D-)
- J8 pad 3: GND -> Net-(J8-D+)
- J8 pad 4: 3V3 -> unconnected-(J8-ID-Pad4)
- Q2 pad 2: /system_SSR_control/SW_ARM -> Net-(Q2-G)
- Q3 pad 2: 3V3 -> +3V3
- Q4 pad 1: 3V3 -> +3V3
- R1 pad 2: /SYS_ENABLE -> /system_SSR_control/SYS_ENABLE
- R11 pad 2: V_BAT -> +BATT
- R12 pad 2: 3V3 -> +3V3
- R13 pad 1: 3V3 -> Net-(U4-A0)
- R13 pad 2: /SCL -> GND
- R14 pad 1: 3V3 -> +3V3
- R14 pad 2: /SDA -> Net-(U4-A0)
- R15 pad 2: 3V3 -> +3V3
- R17 pad 1: /LEDs/red_LED -> +3V3
- R17 pad 2: Net-(J5-Pad4) -> Net-(U4-A1)
- R18 pad 1: /LEDs/green_LED -> Net-(U4-A1)
- R18 pad 2: Net-(J5-Pad6) -> GND
- R19 pad 1: /LEDs/blue_LED -> +3V3
- R19 pad 2: Net-(J5-Pad1) -> Net-(U4-A2)
- R20 pad 1: /LEDs/yellow_LED -> Net-(U4-A2)
- R20 pad 2: Net-(J5-Pad3) -> GND
- R21 pad 1: /LEDs/white_LED -> /Input Headers/PC_TX
- R21 pad 2: Net-(J5-Pad5) -> /Input Headers/VCCIO
- R3 pad 2: 3V3 -> +3V3
- R4 pad 2: 3V3 -> +3V3
- R5 pad 2: V_BAT -> +BATT
- R6 pad 2: /system_SSR_control/SW_ARM -> Net-(Q2-G)
- R7 pad 1: 5V -> +5V
Routing:
- net 5V: track 161.7 -> 0.00 mm
- net 3V3: track 135.8 -> 0.00 mm
- net /system_SSR_control/THR_SSR_P4_COIL-: track 60.3 -> 0.00 mm
- net /THR_KILLED: track 38.2 -> 0.00 mm, vias 1 -> 0
- net /LEDs/white_LED: track 31.4 -> 0.00 mm
- net /LEDs/blue_LED: track 31.2 -> 0.00 mm, vias 1 -> 0
- net /system_SSR_control/SW_ARM: track 28.3 -> 0.00 mm
- net /launchpad_interface/LED_strip: track 26.0 -> 0.00 mm
- net /LEDs/yellow_LED: track 21.8 -> 0.00 mm, vias 1 -> 0
- net /leak_sensor/leak_out: track 20.2 -> 0.00 mm
- net /Input Headers/leak_probe: track 20.1 -> 0.00 mm
- net /SCL: track 18.4 -> 0.00 mm
- net /SDA: track 17.8 -> 0.00 mm
- net /Input Headers/KillSwitchB: track 16.5 -> 0.00 mm, vias 1 -> 0
- net /LEDs/green_LED: track 15.9 -> 0.00 mm, vias 1 -> 0
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- removed copper zone on B.Cu, net GND
- removed copper zone on F.Cu, net GND
- removed copper zone on F.Cu, net Net-(C1-A)
- removed copper zone on F.Cu, net Net-(C2-A)
Other:
- board size 49.8 x 49.8 mm -> 66 x 50.8 mm
- board text removed: "BAT"
- board text removed: "DNP"
- board text removed: "MEB"
- board text removed: "OFF"
- board text removed: "ON"
- board text removed: "THR"
- board text removed: "v1.2"
