File: MEB.kicad_pcb (KiCad board)
At the start: 2 copper layers, 49.8 x 49.8 mm, 45 parts, among them J1 171857-0003, J10 1x4 Header, J2 171856-0002, J3 171857-0003, J4 171856-0002, J5 Header, J6 171856-0002, J7 171857-0003, J8 171856-0004, J9 TLW-104-05-T-D, P1 MSP-EXP430G2ET Interface with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, Q1 2.1V, Q2 2N7000, Q3 2N7000, Q4 TP2104N3-G, SW1 FSM2JSMA, SW2 FSM2JSMA, U1 NCP1117LPST33T3G

Commit message: Fix a variety of small issues
Parts:
- removed F1: 0466002.NRHF, AltiumImport:FP-0466-MFG
- removed G***: LOGO, LOGO
- removed J10: 1x4 Header, AltiumImport:1X4 HEADER
- removed J4: 171856-0002, AltiumImport:SHDR2W99P0X254_1X2_493X635X818P
- removed J7: 171857-0003, AltiumImport:171857-0003
- removed P1: MSP-EXP430G2ET Interface with 1x3 Power Headers, AltiumImport:MSP-EXP430G2ET Interface Power
- removed R13, R14: 4.7k, AltiumImport:SMD-0805-RES
- removed R17, R18, R19, R20, R21: 47, AltiumImport:SMD-0805-RES
- removed R5: 100k, AltiumImport:SMD-0805-RES
- added C4: 12.5p, Capacitor_SMD:C_0805_2012Metric_Pad1.18x1.45mm_HandSolder, F.Cu at (156.5, 101.4)
- added D4: 3.2V, AltiumImport:0805_A, F.Cu at (144.5, 80.3)
- added D5: 3.2V, AltiumImport:0805_A, F.Cu at (144.5, 83.1)
- added D6: 3.2V, AltiumImport:0805_A, F.Cu at (168.0, 103.9)
- added R25: 200, Resistor_SMD:R_0805_2012Metric_Pad1.20x1.40mm_HandSolder, F.Cu at (151.7, 88.8)
- added R26: 20, Resistor_SMD:R_0805_2012Metric_Pad1.20x1.40mm_HandSolder, F.Cu at (163.3, 104.3)
- added U2: MSP430FR2355TPT, SWLib:PT0048A_N, F.Cu at (148.4, 102.7)
- added U3: FT230XS-R, SWLib:SOIC_30XS-R_FTD, F.Cu at (136.3, 90.4)
- added U4: PCT2075DP, Package_SO:TSSOP-8_3x3mm_P0.65mm, F.Cu at (159.6, 121.3)
- C3: value 1uF -> 12.5p; footprint AltiumImport:FP-0603-L_1_6_0_1-W_0_8_0-IPC_A -> Capacitor_SMD:C_0805_2012Metric_Pad1.18x1.45mm_HandSolder
- J5: value Header -> 171856-0004; footprint AltiumImport:2x3 Header -> AltiumImport:SHDR4W99P0X254_1X4_1001X635X1105P
- J6: value 171856-0002 -> 171857-0003; footprint AltiumImport:SHDR2W99P0X254_1X2_493X635X818P -> AltiumImport:171857-0003
- J8: value 171856-0004 -> USB_B_Micro; footprint AltiumImport:SHDR4W99P0X254_1X4_1001X635X1105P -> Connector_USB:USB_Micro-B_GCT_USB3076-30-A
- R1, R11, R12, R2, R3, R4, R6, R7: footprint AltiumImport:SMD-0805-RES -> Resistor_SMD:R_0805_2012Metric_Pad1.20x1.40mm_HandSolder
- R15: footprint AltiumImport:FP-RMCF0805-IPC_C -> Resistor_SMD:R_0805_2012Metric_Pad1.20x1.40mm_HandSolder
- R16: footprint AltiumImport:FP-RNCP0805-IPC_C -> Resistor_SMD:R_0805_2012Metric_Pad1.20x1.40mm_HandSolder
- moved J1 54.6 mm to (127.7, 81.4), turned to 0 degrees
- moved R1 40.5 mm to (151.7, 74.1), turned to 0 degrees
- moved J8 38.1 mm to (137.1, 82.1), turned to 0 degrees
- moved R4 38.1 mm to (151.7, 82.9), turned to 0 degrees
- moved F2 37.7 mm to (151.5, 120.7), turned to 0 degrees
- moved R3 37.7 mm to (151.7, 80.0), turned to 0 degrees
- moved R16 37.5 mm to (164.0, 114.8), turned to 0 degrees
- moved R7 37.5 mm to (151.2, 123.8), turned to 0 degrees
- moved R2 36.4 mm to (151.7, 77.0), turned to 0 degrees
- moved J2 35.4 mm to (142.7, 91.1)
- moved J6 33.9 mm to (136.3, 105.7)
- moved C2 33.7 mm to (145.4, 123.7), turned to 0 degrees
- moved J3 33.2 mm to (127.7, 105.7)
- moved J5 33.0 mm to (125.3, 118.9), turned to 0 degrees
- moved D1 32.4 mm to (163.0, 91.0), turned to 0 degrees
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Connections:
- net /launchpad_interface/leak_out renamed /leak_sensor/leak_out
- net /system_SSR_control/SYS_SW renamed /Input Headers/SYS_OFF
- net Net-(Q2-D) renamed /Input Headers/KillSwitchB
- net Net-(Q4-Gate) renamed /Input Headers/leak_probe
- C3 pad 1: 3V3 -> Net-(U2-P2.6_MCLK_XOUT)
- F2 pad 2: 3V3 -> +3V3
- J3 pad 2: /system_SSR_control/SW_ARM -> unconnected-(J3-Pad2)
- J5 pad 1: Net-(J5-Pad1) -> /Output Headers/I2C_SCL
- J5 pad 2: GND -> /Output Headers/I2C_SDA
- J5 pad 3: Net-(J5-Pad3) -> GND
- J5 pad 4: Net-(J5-Pad4) -> +3V3
- J6 pad 1: V_BAT -> GND
- J6 pad 2: GND -> /Output Headers/LED_Strip
- J8 pad 1: /SCL -> +5V
- J8 pad 2: /SDA -> Net-(J8-D-)
- J8 pad 3: GND -> Net-(J8-D+)
- J8 pad 4: 3V3 -> unconnected-(J8-ID-Pad4)
- Q2 pad 2: /system_SSR_control/SW_ARM -> Net-(Q2-G)
- Q3 pad 2: 3V3 -> +3V3
- Q4 pad 1: 3V3 -> +3V3
- R1 pad 2: /SYS_ENABLE -> /system_SSR_control/SYS_ENABLE
- R11 pad 2: V_BAT -> +BATT
- R12 pad 2: 3V3 -> +3V3
- R15 pad 2: 3V3 -> +3V3
- R3 pad 2: 3V3 -> +3V3
- R4 pad 2: 3V3 -> +3V3
- R6 pad 2: /system_SSR_control/SW_ARM -> Net-(Q2-G)
- R7 pad 1: 5V -> +5V
Routing:
- net 5V: track 161.7 -> 0.00 mm
- net 3V3: track 135.8 -> 0.00 mm
- net /system_SSR_control/THR_SSR_P4_COIL-: track 60.3 -> 0.00 mm
- net GND: track 58.7 -> 0.00 mm, vias 3 -> 0
- net /THR_KILLED: track 38.2 -> 0.00 mm, vias 1 -> 0
- net /LEDs/white_LED: track 31.4 -> 0.00 mm
- net /LEDs/blue_LED: track 31.2 -> 0.00 mm, vias 1 -> 0
- net /system_SSR_control/SW_ARM: track 28.3 -> 0.00 mm
- net /launchpad_interface/LED_strip: track 26.0 -> 0.00 mm
- net /Input Headers/SYS_OFF: track 25.6 -> 0.00 mm
- net /system_SSR_control/SYS_SSR_P4_COIL-: track 25.2 -> 0.00 mm
- net /LEDs/yellow_LED: track 21.8 -> 0.00 mm, vias 1 -> 0
- net /leak_sensor/leak_out: track 20.2 -> 0.00 mm
- net /Input Headers/leak_probe: track 20.1 -> 0.00 mm
- net /SCL: track 18.4 -> 0.00 mm
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- removed copper zone on B.Cu, net GND
- removed copper zone on F.Cu, net GND
- removed copper zone on F.Cu, net Net-(C1-A)
- removed copper zone on F.Cu, net Net-(C2-A)
Other:
- board outline removed
- board text removed: "BAT"
- board text removed: "DNP"
- board text removed: "MEB"
- board text removed: "OFF"
- board text removed: "ON"
- board text removed: "THR"
- board text removed: "v1.2"
