File: LEDs.kicad_sch (KiCad schematic)
At the start: 6 parts, among them J5 Header

Commit message: Cleanup symbol field table
Parts:
- J5: ALTIUM_VALUE 2x3 -> (none); COMPONENTLINK1DESCRIPTION http://www.farnell.com/datasheets/1876884.pdf -> (none); COMPONENTLINK1URL http://www.farnell.com/datasheets/1876884.pdf -> (none); CONTACT PLATING Tin Plated Contacts -> (none); CONTACT TERMINATION TYPE Through Hole -> (none); DESCRIPTION 1 FCI - 67996-406HLF - BOARD-BOARD CONNECTOR HEADER, 6 POSITI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 -> (none); GENDER Header -> (none); MANUFACTURER Amphenol ICC (FCI) -> (none); MANUFACTURER 1 FCI -> (none); MANUFACTURER PART NUMBER 67996-406HLF -> (none); NO. OF CONTACTS 6 -> (none); NO. OF ROWS 2 -> (none); PITCH SPACING 2.54 -> (none); PRICING 1 1=0.254, 10=0.218, 25=0.186, 50=0.178, 100=0.16, 250=0.153,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 -> (none); PRODUCT RANGE BergStik 67996 Series -> (none); Part Number (none) -> 67996-406HLF; ROHS YES -> (none); STOCK 1 441 -> (none); SUPPLIER 1 Newark -> (none); SUPPLIER PART NUMBER 1 20M2191 -> (none)
- R17, R18, R19, R20, R21: @ QTY 1500 -> (none); ALTIUM_VALUE 47 -> (none); COMPOSITION Thick Film -> (none); DATASHEETS http://industrial.panasonic.com/www-cgi/jvcr13pz.cgi?E+PZ+3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 -> (none); DIGI-KEY PART NUMBER P47.0CCT-ND -> (none); FACTORY STOCK 0 -> (none); FAILURE RATE - -> (none); FEATURES Automotive AEC-Q200 -> (none); HEIGHT - SEATED (MAX) 0.028" (0.70mm) -> (none); IMAGE //media.digikey.com/Renders/Panasonic%20Renders/ERJ-0805%20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 -> (none); MANUFACTURER Panasonic Electronic Components -> (none); MANUFACTURER PART NUMBER ERJ-6ENF47R0V -> (none); MINIMUM QUANTITY 1 -> (none); NUMBER OF TERMINATIONS 2 -> (none); OPERATING TEMPERATURE -55°C ~ 155°C -> (none); PACKAGE / CASE 0805 (2012 Metric) -> (none); PACKAGING Cut Tape (CT) -> (none); PART NUMBER ERJ-6ENF47R0V -> (none); PART STATUS Active -> (none); POWER (WATTS) 0.125W, 1/8W -> (none); Part Number (none) -> ERJ-6ENF47R0V; QUANTITY AVAILABLE 66070 -> (none); SERIES ERJ -> (none); SIZE / DIMENSION 0.079" L x 0.049" W (2.00mm x 1.25mm) -> (none); SUPPLIER DEVICE PACKAGE 0805 -> (none); TEMPERATURE COEFFICIENT ±100ppm/°C -> (none); TOLERANCE ±1% -> (none); UNIT PRICE (USD) 0.00729 -> (none)
