File: launchpad_interface.kicad_sch (KiCad schematic)
At the start: 3 parts, among them P1 MSP-EXP430G2ET Interface with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

Commit message: Cleanup symbol field table
Parts:
- P1: LINK * -> (none); MANUFACTURER Texas Instruments -> (none); MANUFACTURER PART NUMBER MSP-EXP430G2ET -> (none); Part Number (none) -> MSP-EXP430G2ET
- R13, R14: ALTIUM_VALUE 4.7k -> (none); DATASHEET LINK https://www.yageo.com/upload/media/product/productsearch/da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 -> (none); MANUFACTURER YAGEO -> (none); MANUFACTURER PART NUMBER RT0805FRE074K7L -> (none); OPERATING TEMPERATURE -55°C ~ 155°C -> (none); PACKAGE / CASE 0805 (2012 Metric) -> (none); Part Number (none) -> RT0805FRE074K7L; ROHS YES -> (none)
Changed lines of the file:
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@@
     (stroke (width 0.254) (type default))
   )
+  (polyline (pts (xy 10.16 132.08) (xy 60.96 208.28))
+    (stroke (width 0.762) (type solid) (color 255 0 0 1))
+  )
   (wire (pts (xy 119.38 119.38) (xy 116.84 119.38))
     (stroke (width 0.254) (type default))
   )
+  (polyline (pts (xy 60.96 132.08) (xy 10.16 208.28))
+    (stroke (width 0.762) (type solid) (color 255 0 0 1))
+  )
   (wire (pts (xy 123.19 48.26) (xy 123.19 50.8))
     (stroke (width 0.254) (type default))
@@
     (fill (type none))
   )
-  (polyline
-    (pts
-      (xy 10.16 132.08)
-      (xy 60.96 208.28)
-    )
-    (stroke (width 0.762) (type solid) (color 255 0 0 1))
-    (fill (type none))
-  )
-  (polyline
-    (pts
-      (xy 60.96 132.08)
-      (xy 10.16 208.28)
-    )
-    (stroke (width 0.762) (type solid) (color 255 0 0 1))
-    (fill (type none))
-  )
   (image (at 69.215 170.8315) (scale 1.33224)
     (data
@@
       (effects (font (size 1.27 1.27)) hide)
     )
-    (property "MANUFACTURER" "YAGEO" (at 42.418 70.612 0)
-      (effects (font (size 1.27 1.27)) (justify left bottom) hide)
-    )
-    (property "ALTIUM_VALUE" "4.7k" (at 42.418 70.612 0)
-      (effects (font (size 1.27 1.27)) (justify left bottom) hide)
-    )
-    (property "OPERATING TEMPERATURE" "-55°C ~ 155°C" (at 42.418 70.612 0)
-      (effects (font (size 1.27 1.27)) (justify left bottom) hide)
-    )
-    (property "PACKAGE / CASE" "0805 (2012 Metric)" (at 42.418 70.612 0)
-      (effects (font (size 1.27 1.27)) (justify left bottom) hide)
-    )
-    (property "MANUFACTURER PART NUMBER" "RT0805FRE074K7L" (at 42.418 70.612 0)
-      (effects (font (size 1.27 1.27)) (justify left bottom) hide)
-    )
-    (property "DATASHEET LINK" "https://www.yageo.com/upload/media/product/productsearch/datasheet/rchip/PYu-RT_1-to-0.01_RoHS_L_12.pdf" (at 42.418 70.612 0)
-      (effects (font (size 1.27 1.27)) (justify left bottom) hide)
-    )
-    (property "ROHS" "YES" (at 42.418 70.612 0)
-      (effects (font (size 1.27 1.27)) (justify left bottom) hide)
+    (property "Part Number" "RT0805FRE074K7L" (at 43.18 76.2 0)
+      (effects (font (size 1.27 1.27)) hide)
     )
     (pin "1")
@@
       (effects (font (size 1.27 1.27)) hide)
     )
-    (property "MANUFACTURER" "YAGEO" (at 50.038 70.612 0)
-      (effects (font (size 1.27 1.27)) (justify left bottom) hide)
-    )
-    (property "ALTIUM_VALUE" "4.7k" (at 50.038 70.612 0)
-      (effects (font (size 1.27 1.27)) (justify left bottom) hide)
-    )
-    (property "OPERATING TEMPERATURE" "-55°C ~ 155°C" (at 50.038 70.612 0)
-      (effects (font (size 1.27 1.27)) (justify left bottom) hide)
-    )
-    (property "PACKAGE / CASE" "0805 (2012 Metric)" (at 50.038 70.612 0)
-      (effects (font (size 1.27 1.27)) (justify left bottom) hide)
-    )
-    (property "MANUFACTURER PART NUMBER" "RT0805FRE074K7L" (at 50.038 70.612 0)
-      (effects (font (size 1.27 1.27)) (justify left bottom) hide)
-    )
-    (property "DATASHEET LINK" "https://www.yageo.com/upload/media/product/productsearch/datasheet/rchip/PYu-RT_1-to-0.01_RoHS_L_12.pdf" (at 50.038 70.612 0)
-      (effects (font (size 1.27 1.27)) (justify left bottom) hide)
-    )
-    (property "ROHS" "YES" (at 50.038 70.612 0)
-      (effects (font (size 1.27 1.27)) (justify left bottom) hide)
+    (property "Part Number" "RT0805FRE074K7L" (at 50.8 76.2 0)
+      (effects (font (size 1.27 1.27)) hide)
     )
     (pin "1")
@@
       (effects (font (size 1.27 1.27)) hide)
     )
-    (property "LINK" "*" (at 79.502 105.41 0)
-      (effects (font (size 1.27 1.27)) (justify left bottom) hide)
-    )
-    (property "MANUFACTURER" "Texas Instruments" (at 76.962 55.372 0)
-      (effects (font (size 1.27 1.27)) (justify left bottom) hide)
-    )
-    (property "MANUFACTURER PART NUMBER" "MSP-EXP430G2ET" (at 76.962 55.372 0)
-      (effects (font (size 1.27 1.27)) (justify left bottom) hide)
-    )
-    (property "ALTIUM_VALUE" "" (at 76.962 55.372 0)
-      (effects (font (size 1.27 1.27)) (justify left bottom) hide)
+    (property "Part Number" "MSP-EXP430G2ET" (at 114.3 83.82 0)
+      (effects (font (size 1.27 1.27)) hide)
     )
     (pin "1")
