File: input_headers.kicad_sch (KiCad schematic)
At the start: 21 parts, among them J1 171857-0003, J2 171856-0002, J7 Conn_01x07, J8 USB_B_Micro, J9 TLW-104-05-T-D, U3 FT230XS-R

Commit message: Fix a variety of small issues
Parts:
- added R5: 0, symbol Device:R_US
- renumbered C5 to C10, C5 to C11, C5 to C12, C5 to C7, C5 to C8, D2 to D4, D2 to D5
Connections:
- net GND: no longer C10.2, C11.2, C12.2, C7.2, C8.2, C9.2, J8.5 (GND), U3.13 (GND)
- net at C12.1, J8.3 (D+), R9.1: now also C11.1, J8.2 (D-), R10.1
- net at J8.6 (Shield): now also R5.1
- new net: C11.2, C12.2, C7.2, C8.2, C9.2, U3.13 (GND)
- new net: C10.2, J8.5 (GND), R5.2
- no-connect marks 0 -> 5
Other:
- moved on the sheet: C11, C12, C7, C8, C9, D4, J1, J2, J7, J9, R21, R22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
