File: mcu_interface.kicad_sch (KiCad schematic)
At the start: 6 parts, among them U2 MSP430FR2355TPT, Y1 32768

Commit message: no changes
Parts:
- C5: footprint (none) -> Capacitor_SMD:C_0805_2012Metric_Pad1.18x1.45mm_HandSolder
- Y1: footprint (none) -> Crystal:Crystal_AT310_D3.0mm_L10.0mm_Horizontal
Changed lines of the file:
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@@
       (effects (font (size 1.27 1.27)) (justify left))
     )
-    (property "Footprint" "" (at 63.1952 80.01 0)
+    (property "Footprint" "Capacitor_SMD:C_0805_2012Metric_Pad1.18x1.45mm_HandSolder" (at 63.1952 80.01 0)
       (effects (font (size 1.27 1.27)) hide)
     )
@@
       (effects (font (size 1.27 1.27)) (justify left))
     )
-    (property "Footprint" "" (at 48.26 124.46 0)
+    (property "Footprint" "Crystal:Crystal_AT310_D3.0mm_L10.0mm_Horizontal" (at 48.26 124.46 0)
       (effects (font (size 1.27 1.27)) hide)
     )

Commit message: Began PCB Design
Parts:
- C6: footprint (none) -> Capacitor_SMD:CP_Elec_4x5.8
Changed lines of the file:
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@@
       (effects (font (size 1.27 1.27)) (justify left))
     )
-    (property "Footprint" "" (at 45.4152 80.01 0)
+    (property "Footprint" "Capacitor_SMD:CP_Elec_4x5.8" (at 45.4152 80.01 0)
       (effects (font (size 1.27 1.27)) hide)
     )
